File: encoder.kicad_sch (KiCad schematic)
At the start: 7 parts, among them SW1 RotaryEncoder_Switch_MP

Commit message: Initial component placement
Parts:
- C1, C2, C3: footprint (none) -> Capacitor_SMD:C_0805_2012Metric_Pad1.18x1.45mm_HandSolder
- R12, R13, R14: footprint (none) -> Resistor_SMD:R_0805_2012Metric_Pad1.20x1.40mm_HandSolder
- SW1: footprint (none) -> Rotary_Encoder:RotaryEncoder_Alps_EC12E-Switch_Vertical_H20mm
Changed lines of the file:
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@@
 			)
 		)
-		(property "Footprint" ""
+		(property "Footprint" "Rotary_Encoder:RotaryEncoder_Alps_EC12E-Switch_Vertical_H20mm"
 			(at 138.43 87.376 0)
 			(effects
@@
 			)
 		)
-		(property "Footprint" ""
+		(property "Footprint" "Capacitor_SMD:C_0805_2012Metric_Pad1.18x1.45mm_HandSolder"
 			(at 125.4252 118.11 0)
 			(effects
@@
 			)
 		)
-		(property "Footprint" ""
+		(property "Footprint" "Resistor_SMD:R_0805_2012Metric_Pad1.20x1.40mm_HandSolder"
 			(at 121.412 128.27 90)
 			(effects
@@
 			)
 		)
-		(property "Footprint" ""
+		(property "Footprint" "Capacitor_SMD:C_0805_2012Metric_Pad1.18x1.45mm_HandSolder"
 			(at 160.9852 102.87 0)
 			(effects
@@
 			)
 		)
-		(property "Footprint" ""
+		(property "Footprint" "Resistor_SMD:R_0805_2012Metric_Pad1.20x1.40mm_HandSolder"
 			(at 149.352 99.06 90)
 			(effects
@@
 			)
 		)
-		(property "Footprint" ""
+		(property "Footprint" "Capacitor_SMD:C_0805_2012Metric_Pad1.18x1.45mm_HandSolder"
 			(at 133.0452 132.08 0)
 			(effects
@@
 			)
 		)
-		(property "Footprint" ""
+		(property "Footprint" "Resistor_SMD:R_0805_2012Metric_Pad1.20x1.40mm_HandSolder"
 			(at 113.792 114.3 90)
 			(effects

Commit message: Initial layout
Parts:
- renumbered C1 to C4, C2 to C5, C3 to C6, R12 to R15, R13 to R16, R14 to R17, SW1 to SW2
Changed lines of the file:
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@@
 		(on_board yes)
 		(dnp no)
-		(property "Reference" "#PWR010"
+		(property "Reference" "#PWR015"
 			(at 151.13 110.49 0)
 			(effects
@@
 		(on_board yes)
 		(dnp no)
-		(property "Reference" "SW1"
+		(property "Reference" "SW2"
 			(at 142.24 81.28 0)
 			(effects
@@
 		(on_board yes)
 		(dnp no)
-		(property "Reference" "C1"
+		(property "Reference" "C4"
 			(at 128.27 113.0299 0)
 			(effects
@@
 		(on_board yes)
 		(dnp no)
-		(property "Reference" "#PWR08"
+		(property "Reference" "#PWR013"
 			(at 123.19 139.7 0)
 			(effects
@@
 		(dnp no)
 		(fields_autoplaced yes)
-		(property "Reference" "#PWR05"
+		(property "Reference" "#PWR012"
 			(at 119.38 86.36 0)
 			(effects
@@
 		(dnp no)
 		(fields_autoplaced yes)
-		(property "Reference" "R13"
+		(property "Reference" "R16"
 			(at 125.73 126.9999 0)
 			(effects
@@
 		(dnp no)
 		(fields_autoplaced yes)
-		(property "Reference" "C3"
+		(property "Reference" "C6"
 			(at 163.83 97.7899 0)
 			(effects
@@
 		(on_board yes)
 		(dnp no)
-		(property "Reference" "#PWR04"
+		(property "Reference" "#PWR07"
 			(at 115.57 125.73 0)
 			(effects
@@
 		(dnp no)
 		(fields_autoplaced yes)
-		(property "Reference" "R14"
+		(property "Reference" "R17"
 			(at 153.67 97.7899 0)
 			(effects
@@
 		(dnp no)
 		(fields_autoplaced yes)
-		(property "Reference" "#PWR09"
+		(property "Reference" "#PWR014"
 			(at 151.13 90.17 0)
 			(effects
@@
 		(dnp no)
 		(fields_autoplaced yes)
-		(property "Reference" "C2"
+		(property "Reference" "C5"
 			(at 135.89 126.9999 0)
 			(effects
@@
 		(dnp no)
 		(fields_autoplaced yes)
-		(property "Reference" "R12"
+		(property "Reference" "R15"
 			(at 118.11 113.0299 0)
 			(effects

Commit message: KiCAD version update
Parts:
- renumbered C4 to C1, C5 to C2, C6 to C3, R15 to R12, R16 to R13, R17 to R14, SW2 to SW1
Changed lines of the file:
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@@
 (kicad_sch
-	(version 20231120)
+	(version 20250114)
 	(generator "eeschema")
-	(generator_version "8.0")
+	(generator_version "9.0")
 	(paper "A4")
 	(junction
@@
 		(on_board yes)
 		(dnp no)
-		(property "Reference" "#PWR015"
+		(property "Reference" "#PWR010"
 			(at 151.13 110.49 0)
 			(effects
@@
 		(on_board yes)
 		(dnp no)
-		(property "Reference" "SW2"
+		(property "Reference" "SW1"
 			(at 142.24 81.28 0)
 			(effects
@@
 		(on_board yes)
 		(dnp no)
-		(property "Reference" "C4"
+		(property "Reference" "C1"
 			(at 128.27 113.0299 0)
 			(effects
@@
 		(on_board yes)
 		(dnp no)
-		(property "Reference" "#PWR013"
+		(property "Reference" "#PWR08"
 			(at 123.19 139.7 0)
 			(effects
@@
 		(dnp no)
 		(fields_autoplaced yes)
-		(property "Reference" "#PWR012"
+		(property "Reference" "#PWR05"
 			(at 119.38 86.36 0)
 			(effects
@@
 		(dnp no)
 		(fields_autoplaced yes)
-		(property "Reference" "R16"
+		(property "Reference" "R13"
 			(at 125.73 126.9999 0)
 			(effects
@@
 		(dnp no)
 		(fields_autoplaced yes)
-		(property "Reference" "C6"
+		(property "Reference" "C3"
 			(at 163.83 97.7899 0)
 			(effects
@@
 		(on_board yes)
 		(dnp no)
-		(property "Reference" "#PWR07"
+		(property "Reference" "#PWR04"
 			(at 115.57 125.73 0)
 			(effects
@@
 		(dnp no)
 		(fields_autoplaced yes)
-		(property "Reference" "R17"
+		(property "Reference" "R14"
 			(at 153.67 97.7899 0)
 			(effects
@@
 		(dnp no)
 		(fields_autoplaced yes)
-		(property "Reference" "#PWR014"
+		(property "Reference" "#PWR09"
 			(at 151.13 90.17 0)
 			(effects
@@
 		(dnp no)
 		(fields_autoplaced yes)
-		(property "Reference" "C5"
+		(property "Reference" "C2"
 			(at 135.89 126.9999 0)
 			(effects
@@
 		(dnp no)
 		(fields_autoplaced yes)
-		(property "Reference" "R15"
+		(property "Reference" "R12"
 			(at 118.11 113.0299 0)
 			(effects

Commit message: Encoder component values
Parts:
- C1, C2, C3: value C -> 100n
- R12, R13, R14: value R -> 10k
Changed lines of the file:
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@@
 	(wire
 		(pts
-			(xy 119.38 82.55) (xy 119.38 91.44)
+			(xy 119.38 88.9) (xy 119.38 91.44)
 		)
 		(stroke
@@
 		(dnp no)
 		(property "Reference" "C1"
-			(at 128.27 113.0299 0)
-			(effects
-				(font
-					(size 1.27 1.27)
-				)
-				(justify left)
-			)
-		)
-		(property "Value" "C"
-			(at 128.27 115.5699 0)
+			(at 126.746 112.268 0)
+			(effects
+				(font
+					(size 1.27 1.27)
+				)
+				(justify left)
+			)
+		)
+		(property "Value" "100n"
+			(at 126.238 116.332 0)
 			(effects
 				(font
@@
 	(symbol
 		(lib_id "power:VCC")
-		(at 119.38 82.55 0)
+		(at 119.38 88.9 0)
 		(unit 1)
 		(exclude_from_sim no)
@@
 		(fields_autoplaced yes)
 		(property "Reference" "#PWR05"
-			(at 119.38 86.36 0)
+			(at 119.38 92.71 0)
 			(effects
 				(font
@@
 		)
 		(property "Value" "VCC"
-			(at 119.38 77.47 0)
+			(at 119.38 83.82 0)
 			(effects
 				(font
@@
 		)
 		(property "Footprint" ""
-			(at 119.38 82.55 0)
+			(at 119.38 88.9 0)
 			(effects
 				(font
@@
 		)
 		(property "Datasheet" ""
-			(at 119.38 82.55 0)
+			(at 119.38 88.9 0)
 			(effects
 				(font
@@
 		)
 		(property "Description" "Power symbol creates a global label with name \"VCC\""
-			(at 119.38 82.55 0)
+			(at 119.38 88.9 0)
 			(effects
 				(font
@@
 		(on_board yes)
 		(dnp no)
-		(fields_autoplaced yes)
 		(property "Reference" "R13"
-			(at 125.73 126.9999 0)
-			(effects
-				(font
-					(size 1.27 1.27)
-				)
-				(justify left)
-			)
-		)
-		(property "Value" "R"
-			(at 125.73 129.5399 0)
+			(at 124.714 127 0)
+			(effects
+				(font
+					(size 1.27 1.27)
+				)
+				(justify left)
+			)
+		)
+		(property "Value" "10k"
+			(at 124.714 129.794 0)
 			(effects
 				(font
@@
 		(on_board yes)
 		(dnp no)
-		(fields_autoplaced yes)
 		(property "Reference" "C3"
-			(at 163.83 97.7899 0)
-			(effects
-				(font
-					(size 1.27 1.27)
-				)
-				(justify left)
-			)
-		)
-		(property "Value" "C"
-			(at 163.83 100.3299 0)
+			(at 160.528 97.028 0)
+			(effects
+				(font
+					(size 1.27 1.27)
+				)
+				(justify left)
+			)
+		)
+		(property "Value" "100n"
+			(at 160.782 101.6 0)
 			(effects
 				(font
@@
 		(on_board yes)
 		(dnp no)
-		(fields_autoplaced yes)
 		(property "Reference" "R14"
-			(at 153.67 97.7899 0)
-			(effects
-				(font
-					(size 1.27 1.27)
-				)
-				(justify left)
-			)
-		)
-		(property "Value" "R"
-			(at 153.67 100.3299 0)
+			(at 152.654 96.774 0)
+			(effects
+				(font
+					(size 1.27 1.27)
+				)
+				(justify left)
+			)
+		)
+		(property "Value" "10k"
+			(at 152.908 101.092 0)
 			(effects
 				(font
@@
 		(on_board yes)
 		(dnp no)
-		(fields_autoplaced yes)
 		(property "Reference" "C2"
-			(at 135.89 126.9999 0)
-			(effects
-				(font
-					(size 1.27 1.27)
-				)
-				(justify left)
-			)
-		)
-		(property "Value" "C"
-			(at 135.89 129.5399 0)
+			(at 134.62 126.492 0)
+			(effects
+				(font
+					(size 1.27 1.27)
+				)
+				(justify left)
+			)
+		)
+		(property "Value" "100n"
+			(at 134.62 130.048 0)
 			(effects
 				(font
@@
 		(on_board yes)
 		(dnp no)
-		(fields_autoplaced yes)
 		(property "Reference" "R12"
-			(at 118.11 113.0299 0)
-			(effects
-				(font
-					(size 1.27 1.27)
-				)
-				(justify left)
-			)
-		)
-		(property "Value" "R"
-			(at 118.11 115.5699 0)
-			(effects
-				(font
+			(at 117.094 112.268 0)
+			(effects
+				(font
+					(size 1.27 1.27)
+				)
+				(justify left)
+			)
+		)
+		(property "Value" "10k"
+			(at 117.094 116.078 0)
+			(effects
+				(font

Commit message: Resolve ERC warnings
Parts:
- renumbered C1 to C301, C2 to C302, C3 to C303, R12 to R301, R13 to R302, R14 to R303, SW1 to SW301
Changed lines of the file:
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@@
-		)
-	)
-	(label "{Encoder}"
-		(at 124.46 74.93 0)
-		(effects
-			(font
-				(size 1.27 1.27)
-			)
-			(justify left bottom)
 		)
 	)
@@
 		)
 	)
-	(hierarchical_label "Encoder"
-		(shape input)
+	(hierarchical_label "{Encoder}"
+		(shape output)
 		(at 121.92 74.93 180)
 		(effects
@@
 		(on_board yes)
 		(dnp no)
-		(property "Reference" "#PWR010"
+		(property "Reference" "#PWR0305"
 			(at 151.13 110.49 0)
 			(effects
@@
 			(project "LifeCounter"
 				(path "/16b3e55a-9d75-49bf-a6fe-25414eb3d7da/8ab23184-7a75-4d74-a7c3-8fc56a0d6372"
-					(reference "#PWR015")
-					(unit 1)
-				)
-				(path "/16b3e55a-9d75-49bf-a6fe-25414eb3d7da/e24d82de-f0b3-40eb-9854-28ed19ab91cc"
-					(reference "#PWR010")
+					(reference "#PWR0405")
+					(unit 1)
+				)
+				(path "/16b3e55a-9d75-49bf-a6fe-25414eb3d7da/e24d82de-f0b3-40eb-9854-28ed19ab91cc"
+					(reference "#PWR0305")
 					(unit 1)
 				)
@@
 		(on_board yes)
 		(dnp no)
-		(property "Reference" "SW1"
+		(property "Reference" "SW301"
 			(at 142.24 81.28 0)
 			(effects
@@
 			(project "LifeCounter"
 				(path "/16b3e55a-9d75-49bf-a6fe-25414eb3d7da/8ab23184-7a75-4d74-a7c3-8fc56a0d6372"
-					(reference "SW2")
-					(unit 1)
-				)
-				(path "/16b3e55a-9d75-49bf-a6fe-25414eb3d7da/e24d82de-f0b3-40eb-9854-28ed19ab91cc"
-					(reference "SW1")
+					(reference "SW401")
+					(unit 1)
+				)
+				(path "/16b3e55a-9d75-49bf-a6fe-25414eb3d7da/e24d82de-f0b3-40eb-9854-28ed19ab91cc"
+					(reference "SW301")
 					(unit 1)
 				)
@@
 		(on_board yes)
 		(dnp no)
-		(property "Reference" "C1"
+		(property "Reference" "C301"
 			(at 126.746 112.268 0)
 			(effects
@@
 			(project "LifeCounter"
 				(path "/16b3e55a-9d75-49bf-a6fe-25414eb3d7da/8ab23184-7a75-4d74-a7c3-8fc56a0d6372"
-					(reference "C4")
-					(unit 1)
-				)
-				(path "/16b3e55a-9d75-49bf-a6fe-25414eb3d7da/e24d82de-f0b3-40eb-9854-28ed19ab91cc"
-					(reference "C1")
+					(reference "C401")
+					(unit 1)
+				)
+				(path "/16b3e55a-9d75-49bf-a6fe-25414eb3d7da/e24d82de-f0b3-40eb-9854-28ed19ab91cc"
+					(reference "C301")
 					(unit 1)
 				)
@@
 		(on_board yes)
 		(dnp no)
-		(property "Reference" "#PWR08"
+		(property "Reference" "#PWR0303"
 			(at 123.19 139.7 0)
 			(effects
@@
 			(project "LifeCounter"
 				(path "/16b3e55a-9d75-49bf-a6fe-25414eb3d7da/8ab23184-7a75-4d74-a7c3-8fc56a0d6372"
-					(reference "#PWR013")
-					(unit 1)
-				)
-				(path "/16b3e55a-9d75-49bf-a6fe-25414eb3d7da/e24d82de-f0b3-40eb-9854-28ed19ab91cc"
-					(reference "#PWR08")
+					(reference "#PWR0403")
+					(unit 1)
+				)
+				(path "/16b3e55a-9d75-49bf-a6fe-25414eb3d7da/e24d82de-f0b3-40eb-9854-28ed19ab91cc"
+					(reference "#PWR0303")
 					(unit 1)
 				)
@@
 		(dnp no)
 		(fields_autoplaced yes)
-		(property "Reference" "#PWR05"
+		(property "Reference" "#PWR0302"
 			(at 119.38 92.71 0)
 			(effects
@@
 			(project "LifeCounter"
 				(path "/16b3e55a-9d75-49bf-a6fe-25414eb3d7da/8ab23184-7a75-4d74-a7c3-8fc56a0d6372"
-					(reference "#PWR012")
-					(unit 1)
-				)
-				(path "/16b3e55a-9d75-49bf-a6fe-25414eb3d7da/e24d82de-f0b3-40eb-9854-28ed19ab91cc"
-					(reference "#PWR05")
+					(reference "#PWR0402")
+					(unit 1)
+				)
+				(path "/16b3e55a-9d75-49bf-a6fe-25414eb3d7da/e24d82de-f0b3-40eb-9854-28ed19ab91cc"
+					(reference "#PWR0302")
 					(unit 1)
 				)
@@
 		(on_board yes)
 		(dnp no)
-		(property "Reference" "R13"
+		(property "Reference" "R302"
 			(at 124.714 127 0)
 			(effects
@@
 			(project "LifeCounter"
 				(path "/16b3e55a-9d75-49bf-a6fe-25414eb3d7da/8ab23184-7a75-4d74-a7c3-8fc56a0d6372"
-					(reference "R16")
-					(unit 1)
-				)
-				(path "/16b3e55a-9d75-49bf-a6fe-25414eb3d7da/e24d82de-f0b3-40eb-9854-28ed19ab91cc"
-					(reference "R13")
+					(reference "R402")
+					(unit 1)
+				)
+				(path "/16b3e55a-9d75-49bf-a6fe-25414eb3d7da/e24d82de-f0b3-40eb-9854-28ed19ab91cc"
+					(reference "R302")
 					(unit 1)
 				)
@@
 		(on_board yes)
 		(dnp no)
-		(property "Reference" "C3"
+		(property "Reference" "C303"
 			(at 160.528 97.028 0)
 			(effects
@@
 			(project "LifeCounter"
 				(path "/16b3e55a-9d75-49bf-a6fe-25414eb3d7da/8ab23184-7a75-4d74-a7c3-8fc56a0d6372"
-					(reference "C6")
-					(unit 1)
-				)
-				(path "/16b3e55a-9d75-49bf-a6fe-25414eb3d7da/e24d82de-f0b3-40eb-9854-28ed19ab91cc"
-					(reference "C3")
+					(reference "C403")
+					(unit 1)
+				)
+				(path "/16b3e55a-9d75-49bf-a6fe-25414eb3d7da/e24d82de-f0b3-40eb-9854-28ed19ab91cc"
+					(reference "C303")
 					(unit 1)
 				)
@@
 		(on_board yes)
 		(dnp no)
-		(property "Reference" "#PWR04"
+		(property "Reference" "#PWR0301"
 			(at 115.57 125.73 0)
 			(effects
@@
 			(project "LifeCounter"
 				(path "/16b3e55a-9d75-49bf-a6fe-25414eb3d7da/8ab23184-7a75-4d74-a7c3-8fc56a0d6372"
-					(reference "#PWR07")
-					(unit 1)
-				)
-				(path "/16b3e55a-9d75-49bf-a6fe-25414eb3d7da/e24d82de-f0b3-40eb-9854-28ed19ab91cc"
-					(reference "#PWR04")
+					(reference "#PWR0401")
+					(unit 1)
+				)
+				(path "/16b3e55a-9d75-49bf-a6fe-25414eb3d7da/e24d82de-f0b3-40eb-9854-28ed19ab91cc"
+					(reference "#PWR0301")
 					(unit 1)
 				)
@@
 		(on_board yes)
 		(dnp no)
-		(property "Reference" "R14"
+		(property "Reference" "R303"
 			(at 152.654 96.774 0)
 			(effects
@@
 			(project "LifeCounter"
 				(path "/16b3e55a-9d75-49bf-a6fe-25414eb3d7da/8ab23184-7a75-4d74-a7c3-8fc56a0d6372"
-					(reference "R17")
-					(unit 1)
-				)
-				(path "/16b3e55a-9d75-49bf-a6fe-25414eb3d7da/e24d82de-f0b3-40eb-9854-28ed19ab91cc"
-					(reference "R14")
+					(reference "R403")
+					(unit 1)
+				)
+				(path "/16b3e55a-9d75-49bf-a6fe-25414eb3d7da/e24d82de-f0b3-40eb-9854-28ed19ab91cc"
+					(reference "R303")
 					(unit 1)
 				)
@@
 		(dnp no)
 		(fields_autoplaced yes)
-		(property "Reference" "#PWR09"
+		(property "Reference" "#PWR0304"
 			(at 151.13 90.17 0)
 			(effects
@@
 			(project "LifeCounter"
 				(path "/16b3e55a-9d75-49bf-a6fe-25414eb3d7da/8ab23184-7a75-4d74-a7c3-8fc56a0d6372"
-					(reference "#PWR014")
-					(unit 1)
-				)
-				(path "/16b3e55a-9d75-49bf-a6fe-25414eb3d7da/e24d82de-f0b3-40eb-9854-28ed19ab91cc"
-					(reference "#PWR09")
+					(reference "#PWR0404")
+					(unit 1)
+				)
+				(path "/16b3e55a-9d75-49bf-a6fe-25414eb3d7da/e24d82de-f0b3-40eb-9854-28ed19ab91cc"
+					(reference "#PWR0304")
 					(unit 1)
 				)
@@
 		(on_board yes)
 		(dnp no)
-		(property "Reference" "C2"
+		(property "Reference" "C302"
 			(at 134.62 126.492 0)
 			(effects
@@
 			(project "LifeCounter"
 				(path "/16b3e55a-9d75-49bf-a6fe-25414eb3d7da/8ab23184-7a75-4d74-a7c3-8fc56a0d6372"
-					(reference "C5")
-					(unit 1)
-				)
-				(path "/16b3e55a-9d75-49bf-a6fe-25414eb3d7da/e24d82de-f0b3-40eb-9854-28ed19ab91cc"
-					(reference "C2")
+					(reference "C402")
+					(unit 1)
+				)
+				(path "/16b3e55a-9d75-49bf-a6fe-25414eb3d7da/e24d82de-f0b3-40eb-9854-28ed19ab91cc"
+					(reference "C302")
 					(unit 1)
 				)
@@
 		(on_board yes)
 		(dnp no)
-		(property "Reference" "R12"
+		(property "Reference" "R301"
 			(at 117.094 112.268 0)
 			(effects
@@
 			(project "LifeCounter"
 				(path "/16b3e55a-9d75-49bf-a6fe-25414eb3d7da/8ab23184-7a75-4d74-a7c3-8fc56a0d6372"
-					(reference "R15")
-					(unit 1)
-				)
-				(path "/16b3e55a-9d75-49bf-a6fe-25414eb3d7da/e24d82de-f0b3-40eb-9854-28ed19ab91cc"
-					(reference "R12")
-					(unit 1)
-				)
+					(reference "R401")
+					(unit 1)
+				)
+				(path "/16b3e55a-9d75-49bf-a6fe-25414eb3d7da/e24d82de-f0b3-40eb-9854-28ed19ab91cc"
+					(reference "R301")
+					(unit 1)
+				)

Commit message: Add Testpoints
Parts:
- added TP10: B, symbol Connector:TestPoint
- added TP6: BTN, symbol Connector:TestPoint
- added TP8: A, symbol Connector:TestPoint
Connections:
- net A: now also TP8.1
- net B: now also TP10.1
- net BTN: now also TP6.1

Commit message: Footprint selection
Parts:
- C301, C302, C303: footprint Capacitor_SMD:C_0805_2012Metric_Pad1.18x1.45mm_HandSolder -> Capacitor_SMD:C_1206_3216Metric_Pad1.33x1.80mm_HandSolder
- R301, R302, R303: footprint Resistor_SMD:R_0805_2012Metric_Pad1.20x1.40mm_HandSolder -> Resistor_SMD:R_1206_3216Metric_Pad1.30x1.75mm_HandSolder
- TP10, TP6, TP8: footprint (none) -> TestPoint:TestPoint_Pad_D1.0mm
Changed lines of the file:
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@@
 			)
 		)
-		(property "Footprint" ""
+		(property "Footprint" "TestPoint:TestPoint_Pad_D1.0mm"
 			(at 143.51 123.19 0)
 			(effects
@@
 			)
 		)
-		(property "Footprint" ""
+		(property "Footprint" "TestPoint:TestPoint_Pad_D1.0mm"
 			(at 160.02 93.98 0)
 			(effects
@@
 			)
 		)
-		(property "Footprint" "Capacitor_SMD:C_0805_2012Metric_Pad1.18x1.45mm_HandSolder"
+		(property "Footprint" "Capacitor_SMD:C_1206_3216Metric_Pad1.33x1.80mm_HandSolder"
 			(at 125.4252 118.11 0)
 			(effects
@@
 			)
 		)
-		(property "Footprint" "Resistor_SMD:R_0805_2012Metric_Pad1.20x1.40mm_HandSolder"
+		(property "Footprint" "Resistor_SMD:R_1206_3216Metric_Pad1.30x1.75mm_HandSolder"
 			(at 121.412 128.27 90)
 			(effects
@@
 			)
 		)
-		(property "Footprint" "Capacitor_SMD:C_0805_2012Metric_Pad1.18x1.45mm_HandSolder"
+		(property "Footprint" "Capacitor_SMD:C_1206_3216Metric_Pad1.33x1.80mm_HandSolder"
 			(at 160.9852 102.87 0)
 			(effects
@@
 			)
 		)
-		(property "Footprint" "Resistor_SMD:R_0805_2012Metric_Pad1.20x1.40mm_HandSolder"
+		(property "Footprint" "Resistor_SMD:R_1206_3216Metric_Pad1.30x1.75mm_HandSolder"
 			(at 149.352 99.06 90)
 			(effects
@@
 			)
 		)
-		(property "Footprint" ""
+		(property "Footprint" "TestPoint:TestPoint_Pad_D1.0mm"
 			(at 142.24 109.22 0)
 			(effects
@@
 			)
 		)
-		(property "Footprint" "Capacitor_SMD:C_0805_2012Metric_Pad1.18x1.45mm_HandSolder"
+		(property "Footprint" "Capacitor_SMD:C_1206_3216Metric_Pad1.33x1.80mm_HandSolder"
 			(at 133.0452 132.08 0)
 			(effects
@@
 			)
 		)
-		(property "Footprint" "Resistor_SMD:R_0805_2012Metric_Pad1.20x1.40mm_HandSolder"
+		(property "Footprint" "Resistor_SMD:R_1206_3216Metric_Pad1.30x1.75mm_HandSolder"
 			(at 113.792 114.3 90)
 			(effects
